File: CartesElec/CartePrincipaleR1/CartePrincipaleR1.kicad_pcb (KiCad board)
At the start: 2 copper layers, 100 x 100 mm, 27 parts, among them U1 LT1129-3.3_SOT223

Commit message: Changement mineur
Parts:
- moved NappePompe 0.20 mm to (106.6, 126.6)
Changed lines of the file:
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@@
   )
   (footprint "Connector_IDC:IDC-Header_2x08_P2.54mm_Vertical" (layer "F.Cu")
-    (at 106.6 126.8 -90)
+    (at 106.6 126.6 -90)
     (descr "Through hole IDC box header, 2x08, 2.54mm pitch, DIN 41651 / IEC 60603-13, double rows, https://docs.google.com/spreadsheets/d/16SsEcesNF15N3Lb4niX7dcUr-NY5_MFPQhobNuNppn4/edit#gid=0")
     (tags "Through hole vertical IDC box header THT 2x08 2.54mm double row")
@@
     (effects (font (size 2 2.5) (thickness 0.3)))
   )
-  (gr_text "-" (at 107 132.1 180) (layer "F.SilkS")
+  (gr_text "-" (at 106.8 133.9 180) (layer "F.SilkS")
     (effects (font (size 1 1) (thickness 0.15)))
   )
@@
     (effects (font (size 1 1) (thickness 0.15)))
   )
-  (gr_text "+\n" (at 103.9 131.9 180) (layer "F.SilkS")
+  (gr_text "+\n" (at 104 133.8 180) (layer "F.SilkS")
     (effects (font (size 1 1) (thickness 0.15)))
   )

Commit message: relecture
Parts:
- Nucleo L476RG: renamed from Nucléo L476RG
Changed lines of the file:
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@@
   )
   (paper "A4")
+  (title_block
+    (comment 4 "AISLER Project ID: FQXJOFHD")
+  )
   (layers
     (0 "F.Cu" signal)
@@
     (fp_line (start 1 -0.625) (end 1 0.625) (layer "F.Fab") (width 0.1))
     (fp_line (start -1 0.625) (end -1 -0.625) (layer "F.Fab") (width 0.1))
-    (pad "1" smd roundrect (at -0.9125 0 90) (size 1.025 1.4) (layers "F.Cu" "F.Paste" "F.Mask") (roundrect_rratio 0.243902)
+    (pad "1" smd roundrect (at -0.9125 0 90) (size 1.025 1.4) (layers "F.Cu" "F.Paste" "F.Mask") (roundrect_rratio 0.243902439)
       (net 3 "+3V3") (pintype "passive"))
-    (pad "2" smd roundrect (at 0.9125 0 90) (size 1.025 1.4) (layers "F.Cu" "F.Paste" "F.Mask") (roundrect_rratio 0.243902)
+    (pad "2" smd roundrect (at 0.9125 0 90) (size 1.025 1.4) (layers "F.Cu" "F.Paste" "F.Mask") (roundrect_rratio 0.243902439)
       (net 41 "SDA_I2C1") (pintype "passive"))
     (model "${KICAD6_3DMODEL_DIR}/Resistor_SMD.3dshapes/R_0805_2012Metric.wrl"
@@
     (fp_line (start 1 -0.625) (end 1 0.625) (layer "F.Fab") (width 0.1))
     (fp_line (start -1 0.625) (end -1 -0.625) (layer "F.Fab") (width 0.1))
-    (pad "1" smd roundrect (at -0.9125 0 180) (size 1.025 1.4) (layers "F.Cu" "F.Paste" "F.Mask") (roundrect_rratio 0.243902)
+    (pad "1" smd roundrect (at -0.9125 0 180) (size 1.025 1.4) (layers "F.Cu" "F.Paste" "F.Mask") (roundrect_rratio 0.243902439)
       (net 3 "+3V3") (pintype "passive"))
-    (pad "2" smd roundrect (at 0.9125 0 180) (size 1.025 1.4) (layers "F.Cu" "F.Paste" "F.Mask") (roundrect_rratio 0.243902)
+    (pad "2" smd roundrect (at 0.9125 0 180) (size 1.025 1.4) (layers "F.Cu" "F.Paste" "F.Mask") (roundrect_rratio 0.243902439)
       (net 7 "SCL_I2C3") (pintype "passive"))
     (model "${KICAD6_3DMODEL_DIR}/Resistor_SMD.3dshapes/R_0805_2012Metric.wrl"
@@
     (property "Sheetname" "")
     (attr through_hole)
-    (fp_text reference "Nucléo L476RG" (at 1.7 13.6 180) (layer "F.SilkS")
+    (fp_text reference "Nucleo L476RG" (at 1.7 13.6 180) (layer "F.SilkS")
       (effects (font (size 1 1) (thickness 0.15)))
     )
@@
     (fp_line (start -1 0.625) (end -1 -0.625) (layer "F.Fab") (width 0.1))
     (fp_line (start 1 -0.625) (end 1 0.625) (layer "F.Fab") (width 0.1))
-    (pad "1" smd roundrect (at -0.9125 0 270) (size 1.025 1.4) (layers "F.Cu" "F.Paste" "F.Mask") (roundrect_rratio 0.243902)
+    (pad "1" smd roundrect (at -0.9125 0 270) (size 1.025 1.4) (layers "F.Cu" "F.Paste" "F.Mask") (roundrect_rratio 0.243902439)
       (net 2 "GND") (pintype "passive"))
-    (pad "2" smd roundrect (at 0.9125 0 270) (size 1.025 1.4) (layers "F.Cu" "F.Paste" "F.Mask") (roundrect_rratio 0.243902)
+    (pad "2" smd roundrect (at 0.9125 0 270) (size 1.025 1.4) (layers "F.Cu" "F.Paste" "F.Mask") (roundrect_rratio 0.243902439)
       (net 37 "A_Resistance") (pintype "passive"))
     (model "${KICAD6_3DMODEL_DIR}/Resistor_SMD.3dshapes/R_0805_2012Metric.wrl"
@@
     (fp_line (start -1.98 10.94) (end -3.18 10.94) (layer "F.Fab") (width 0.1))
     (fp_line (start -3.18 6.84) (end -1.98 6.84) (layer "F.Fab") (width 0.1))
-    (pad "1" thru_hole roundrect (at 0 0 270) (size 1.7 1.7) (drill 1) (layers *.Cu *.Mask) (roundrect_rratio 0.147059)
+    (pad "1" thru_hole roundrect (at 0 0 270) (size 1.7 1.7) (drill 1) (layers *.Cu *.Mask) (roundrect_rratio 0.1470588235)
       (net 2 "GND") (pinfunction "Pin_1") (pintype "passive"))
     (pad "2" thru_hole circle (at 2.54 0 270) (size 1.7 1.7) (drill 1) (layers *.Cu *.Mask)
@@
     (fp_line (start 4.52 -3.91) (end 4.52 21.69) (layer "F.Fab") (width 0.1))
     (fp_line (start 5.72 -5.1) (end 5.72 22.88) (layer "F.Fab") (width 0.1))
-    (pad "1" thru_hole roundrect (at 0 0) (size 1.7 1.7) (drill 1) (layers *.Cu *.Mask) (roundrect_rratio 0.147059)
+    (pad "1" thru_hole roundrect (at 0 0) (size 1.7 1.7) (drill 1) (layers *.Cu *.Mask) (roundrect_rratio 0.1470588235)
       (net 2 "GND") (pinfunction "Pin_1") (pintype "passive"))
     (pad "2" thru_hole circle (at 2.54 0) (size 1.7 1.7) (drill 1) (layers *.Cu *.Mask)
@@
     (fp_line (start -1 0.625) (end -1 -0.625) (layer "F.Fab") (width 0.1))
     (fp_line (start 1 0.625) (end -1 0.625) (layer "F.Fab") (width 0.1))
-    (pad "1" smd roundrect (at -0.9125 0 90) (size 1.025 1.4) (layers "F.Cu" "F.Paste" "F.Mask") (roundrect_rratio 0.243902)
+    (pad "1" smd roundrect (at -0.9125 0 90) (size 1.025 1.4) (layers "F.Cu" "F.Paste" "F.Mask") (roundrect_rratio 0.243902439)
       (net 3 "+3V3") (pintype "passive"))
-    (pad "2" smd roundrect (at 0.9125 0 90) (size 1.025 1.4) (layers "F.Cu" "F.Paste" "F.Mask") (roundrect_rratio 0.243902)
+    (pad "2" smd roundrect (at 0.9125 0 90) (size 1.025 1.4) (layers "F.Cu" "F.Paste" "F.Mask") (roundrect_rratio 0.243902439)
       (net 42 "SCL_I2C1") (pintype "passive"))
     (model "${KICAD6_3DMODEL_DIR}/Resistor_SMD.3dshapes/R_0805_2012Metric.wrl"
@@
     (fp_line (start -1 0.625) (end -1 -0.625) (layer "F.Fab") (width 0.1))
     (fp_line (start 1 -0.625) (end 1 0.625) (layer "F.Fab") (width 0.1))
-    (pad "1" smd roundrect (at -0.9125 0 180) (size 1.025 1.4) (layers "F.Cu" "F.Paste" "F.Mask") (roundrect_rratio 0.243902)
+    (pad "1" smd roundrect (at -0.9125 0 180) (size 1.025 1.4) (layers "F.Cu" "F.Paste" "F.Mask") (roundrect_rratio 0.243902439)
       (net 3 "+3V3") (pintype "passive"))
-    (pad "2" smd roundrect (at 0.9125 0 180) (size 1.025 1.4) (layers "F.Cu" "F.Paste" "F.Mask") (roundrect_rratio 0.243902)
+    (pad "2" smd roundrect (at 0.9125 0 180) (size 1.025 1.4) (layers "F.Cu" "F.Paste" "F.Mask") (roundrect_rratio 0.243902439)
       (net 6 "SDA_I2C3") (pintype "passive"))
     (model "${KICAD6_3DMODEL_DIR}/Resistor_SMD.3dshapes/R_0805_2012Metric.wrl"
@@
   (segment (start 147.78 67.68) (end 147.78 65.9) (width 1) (layer "B.Cu") (net 2))
   (segment (start 61.13 115.3) (end 60.93 115.1) (width 0.8) (layer "B.Cu") (net 2))
-  (segment (start 135.1 123.8) (end 133.5 125.4) (width 0.8) (layer "B.Cu") (net 2))
   (segment (start 130.13 129.34) (end 131 128.47) (width 0.8) (layer "B.Cu") (net 2))
   (segment (start 76.68 81.1) (end 72.89 77.31) (width 0.8) (layer "B.Cu") (net 2))
   (segment (start 89.75 87.05) (end 106.6 103.9) (width 0.8) (layer "B.Cu") (net 2))
+  (segment (start 133.27 125.63) (end 133.27 126.2) (width 0.8) (layer "B.Cu") (net 2))
   (segment (start 148.67 78.43) (end 148.67 80.73) (width 0.8) (layer "B.Cu") (net 2))
   (segment (start 148.67 68.57) (end 147.78 67.68) (width 1) (layer "B.Cu") (net 2))
@@
   (segment (start 106.6 129.34) (end 130.13 129.34) (width 0.8) (layer "B.Cu") (net 2))
   (segment (start 147.78 56.71) (end 147.27 56.2) (width 1) (layer "B.Cu") (net 2))
-  (segment (start 133.5 126.2) (end 133.27 126.2) (width 0.8) (layer "B.Cu") (net 2))
   (segment (start 71.9 76) (end 69.2 76) (width 0.4) (layer "B.Cu") (net 2))
   (segment (start 148.67 80.73) (end 148.87 80.93) (width 0.8) (layer "B.Cu") (net 2))
+  (segment (start 135.1 123.8) (end 133.27 125.63) (width 0.8) (layer "B.Cu") (net 2))
   (segment (start 106.6 129.34) (end 106.6 126.8) (width 0.8) (layer "B.Cu") (net 2))
   (segment (start 89.45 87.05) (end 89.75 87.05) (width 0.8) (layer "B.Cu") (net 2))
@@
   (segment (start 148.14 80.2) (end 145.6 80.2) (width 0.8) (layer "B.Cu") (net 2))
   (segment (start 133.27 126.2) (end 131 128.47) (width 0.8) (layer "B.Cu") (net 2))
-  (segment (start 133.5 125.4) (end 133.5 126.2) (width 0.8) (layer "B.Cu") (net 2))
   (segment (start 69.2 76) (end 67.47 74.27) (width 0.8) (layer "B.Cu") (net 2))
   (segment (start 131.31 79.85) (end 129.65 79.85) (width 0.8) (layer "B.Cu") (net 2))
