File: CartesElec/CartePrincipaleR1/CarteSecondaire.kicad_pcb (KiCad board)
At the start: 2 copper layers, 52 x 66 mm, 40 parts, among them J18 Conn_02x08_Top_Bottom, Q1 IRLML0030, Q2 IRLML0030, Q3 IRLML0030, Q4 IRLML0030

Commit message: update carte sec
Parts:
- moved NAPPE2 1.93 mm to (111.8, 179.1)
- renumbered J18 to NAPPE
Routing:
- net CONTACTEUR2_GPIO: track 17.7 -> 20.8 mm
- net DataAX12_TX: track 42.5 -> 40.5 mm
- net CONTACTEUR1_GPIO: track 14.4 -> 16.3 mm
- net +5V: track 162.8 -> 161.1 mm
- net GND: track 260.5 -> 262.1 mm
- net MC2A: track 14.1 -> 14.9 mm
- net RC_2B: track 10.7 -> 11.5 mm
- net MC1B: track 11.2 -> 10.4 mm
- net RC_2A: track 11.2 -> 12.0 mm
- net MC2B: track 7.92 -> 8.72 mm
Other:
- board text added: "3.3V"
- board text added: "5V"
- board text added: "CODEUR"
- board text added: "Carte base roulante"
- board text added: "DIR ="
- board text added: "EV"
- board text added: "Février 2022"
- board text added: "GND"
- board text added: "IO"
- board text added: "Jonathan"
- board text added: "MC"
- board text added: "PUMP"
- board text added: "PWM"
- board text added: "S1"
- board text added: "S2"
- board text added: "S3"
- board text added: "TX"

Commit message: cartePrincipale Update
Parts:
- moved R 0.18 mm to (94.5, 182.1)
- moved R 0.10 mm to (136.5, 126.3)
- moved R 0.10 mm to (94.5, 126.3)
- moved R 0.06 mm to (136.5, 182.3)
Changed lines of the file:
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@@
   )
   (footprint "MountingHole:MountingHole_3.2mm_M3" (layer "F.Cu")
-    (at 94.539011 126.391511)
+    (at 94.5 126.3)
     (descr "Mounting Hole 3.2mm, no annular, M3")
     (tags "mounting hole 3.2mm no annular m3")
@@
   )
   (footprint "MountingHole:MountingHole_3.2mm_M3" (layer "F.Cu")
-    (at 94.539011 182.271511)
+    (at 94.5 182.1)
     (descr "Mounting Hole 3.2mm, no annular, M3")
     (tags "mounting hole 3.2mm no annular m3")
@@
   )
   (footprint "MountingHole:MountingHole_3.2mm_M3" (layer "F.Cu")
-    (at 136.449011 126.391511)
+    (at 136.5 126.3)
     (descr "Mounting Hole 3.2mm, no annular, M3")
     (tags "mounting hole 3.2mm no annular m3")
@@
   )
   (footprint "MountingHole:MountingHole_3.2mm_M3" (layer "F.Cu")
-    (at 136.449011 182.271511)
+    (at 136.5 182.3)
     (descr "Mounting Hole 3.2mm, no annular, M3")
     (tags "mounting hole 3.2mm no annular m3")
